File: 1/1.kicad_sch (KiCad schematic)
At the start: 19 parts, among them J1 Power, J2 Digital/PWM, J3 Analog, J4 Digital/PWM, J5 HC-05, U2 LTC1050

Commit message: Modifactions on kicad project and ltspice are added
Parts:
- removed Entree_Sin1: Conn_01x02, Connector_PinSocket_2.54mm:PinSocket_1x02_P2.54mm_Vertical, symbol Connector_Generic:Conn_01x02
Connections:
- net *5: no longer Capteur1.1 (Pin_1), R5.1
- new net: Capteur1.1 (Pin_1), R5.1
Changed lines of the file:
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@@
-	)
-	(junction
-		(at 156.21 144.78)
-		(diameter 0)
-		(color 0 0 0 0)
 	)
 	(junction
@@
 	)
 	(junction
-		(at 143.51 137.16)
-		(diameter 0)
-		(color 0 0 0 0)
-	)
-	(junction
 		(at 224.79 120.65)
 		(diameter 0)
@@
 	)
 	(junction
-		(at 135.89 137.16)
-		(diameter 0)
-		(color 0 0 0 0)
-	)
-	(junction
 		(at 201.93 120.65)
 		(diameter 0)
@@
 	(wire
 		(pts
-			(xy 135.89 137.16) (xy 143.51 137.16)
-		)
-		(stroke
-			(width 0)
-			(type default)
-		)
-	)
-	(wire
-		(pts
 			(xy 72.39 90.17) (xy 85.09 90.17)
 		)
@@
 	(wire
 		(pts
-			(xy 133.35 137.16) (xy 135.89 137.16)
-		)
-		(stroke
-			(width 0)
-			(type default)
-		)
-	)
-	(wire
-		(pts
 			(xy 156.21 144.78) (xy 166.37 144.78)
 		)
@@
 	(wire
 		(pts
-			(xy 133.35 144.78) (xy 156.21 144.78)
-		)
-		(stroke
-			(width 0)
-			(type default)
-		)
-	)
-	(wire
-		(pts
 			(xy 72.39 57.15) (xy 74.93 57.15)
 		)
@@
 	(wire
 		(pts
-			(xy 134.62 135.89) (xy 135.89 135.89)
-		)
-		(stroke
-			(width 0)
-			(type default)
-		)
-	)
-	(wire
-		(pts
 			(xy 146.05 104.14) (xy 146.05 107.95)
 		)
@@
 	(wire
 		(pts
-			(xy 135.89 135.89) (xy 135.89 137.16)
-		)
-		(stroke
-			(width 0)
-			(type default)
-		)
-	)
-	(wire
-		(pts
 			(xy 175.26 137.16) (xy 175.26 125.73)
 		)
@@
 			(width 0)
 			(type solid)
-		)
-	)
-	(wire
-		(pts
-			(xy 133.35 139.7) (xy 133.35 144.78)
-		)
-		(stroke
-			(width 0)
-			(type default)
 		)
 	)
@@
 	(label "*10"
 		(at 85.09 67.31 180)
-		(effects
-			(font
-				(size 1.27 1.27)
-			)
-			(justify right bottom)
-		)
-	)
-	(label "*5"
-		(at 134.62 135.89 180)
 		(effects
 			(font
@@
 					(unit 1)
 				)
-			)
-		)
-	)
-	(symbol
-		(lib_id "Connector_Generic:Conn_01x02")
-		(at 128.27 139.7 180)
-		(unit 1)
-		(exclude_from_sim yes)
-		(in_bom yes)
-		(on_board yes)
-		(dnp no)
-		(fields_autoplaced yes)
-		(property "Reference" "Entree_Sin1"
-			(at 128.27 130.81 0)
-			(effects
-				(font
-					(size 1.27 1.27)
-				)
-			)
-		)
-		(property "Value" "Conn_01x02"
-			(at 128.27 133.35 0)
-			(effects
-				(font
-					(size 1.27 1.27)
-				)
-			)
-		)
-		(property "Footprint" "Connector_PinSocket_2.54mm:PinSocket_1x02_P2.54mm_Vertical"
-			(at 128.27 139.7 0)
-			(effects
-				(font
-					(size 1.27 1.27)
-				)
-				(hide yes)
-			)
-		)
-		(property "Datasheet" "~"
-			(at 128.27 139.7 0)
-			(effects
-				(font
-					(size 1.27 1.27)
-				)
-				(hide yes)
-			)
-		)
-		(property "Description" ""
-			(at 128.27 139.7 0)
-			(effects
-				(font
-					(size 1.27 1.27)
-				)
-			)
-		)
-		(pin "1"
-		)
-		(pin "2"
-		)
-		(instances
-			(project "1"
-				(path "/e63e39d7-6ac0-4ffd-8aa3-1841a4541b55"
-					(reference "Entree_Sin1")
-					(unit 1)
-				)

Commit message: Rajout des capteurs
Parts:
- removed R2: 1k, Resistor_THT:R_Axial_DIN0207_L6.3mm_D2.5mm_P10.16mm_Horizontal, symbol Device:R
- added Encodeur1: ~, symbol Ma_Library:encodeur
- added Flex_Sensor1: ~, symbol Ma_Library:Flex_Sensor
- added R7: 10k, Resistor_THT:R_Axial_DIN0207_L6.3mm_D2.5mm_P10.16mm_Horizontal, symbol Device:R
- added Servo_Moteur1: ~, symbol Ma_Library:Servo_Moteur
- added U3: ~, symbol Ma_Library:Potentiomètre
Connections:
- net +5V: now also Encodeur1.2 (+), Flex_Sensor1.1 (VCC), Servo_Moteur1.1 (VCC)
- net A1: now also Flex_Sensor1.2 (A1), R7.2
- net GND: now also Encodeur1.1 (GND), R7.1, Servo_Moteur1.2 (GND), U3.5 (A), U3.6 (W)
- net R2: now reaches C4.2, R3.2, U2.3 (+)
- net R2: now also U3.7 (B)
- net *10 renamed CS
- net CS: now also U3.1 (CS)
- net *11 renamed SI
- net SI: now also U3.3 (SI)
- net *3 renamed D3
- net D3: now also Servo_Moteur1.3 (-3); no longer J5.5 (Rx)
- net *5 renamed SW
- net SW: now also Encodeur1.3 (SW)
- net 13 renamed SCK
- net SCK: now also U3.2 (SCK)
- net 2 renamed CLK
- net CLK: now also Encodeur1.5 (CLK); no longer J5.4 (Tx)
- net 4 renamed DATA
- net DATA: now also Encodeur1.4 (DATA)
- net 7 renamed TXD
- net TXD: now also J5.4 (Tx)
- net 8 renamed RXD
- net RXD: now also J5.5 (Rx)
- net SCL/A5 renamed SCL
- net SDA/A4 renamed A4
- no-connect marks 22 -> 12
Other:
- note added: "Opérateurs CAO: Binôme MOSH Maelys/Artur 2025 INSA Toulouse"
- note added: "Projet capteur"

Commit message: Face avant v1
Parts:
- Encodeur1: footprint (none) -> projet_capteur_artur:Encodeur
- Flex_Sensor1: footprint (none) -> projet_capteur_artur:flex_sensor
- Servo_Moteur1: footprint (none) -> projet_capteur_artur:servo
- renumbered U3 to Potentiomètre3
Connections:
- net +5V: now also Potentiomètre3.8 (VDD)
- net 12: now also D1.2 (A)
- net DATA: no longer D1.2 (A)
- net GND: now also Potentiomètre3.4 (VSS)
- no-connect marks 12 -> 10
Other:
- moved on the sheet: J5

Commit message: MAJ de la face arrière avant la routage
Parts:
- Potentiomètre3: footprint (none) -> projet_capteur_artur:potentiometre_digit
Changed lines of the file:
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@@
 	(text_box "Modules"
 		(exclude_from_sim no)
-		(at 39.37 22.86 0)
+		(at 118.11 25.4 0)
 		(size 149.86 57.15)
 		(margins 0.9525 0.9525 0.9525 0.9525)
@@
 			)
 		)
-		(property "Footprint" ""
+		(property "Footprint" "projet_capteur_artur:potentiometre_digit"
 			(at 233.68 57.15 0)
 			(effects

Commit message: Rootage v1
Parts:
- R6: value R -> 320
- renumbered U2 to LTC1050_1, Potentiomètre3 to Potent3
Connections:
- net *6: now also Servo_Moteur1.3 (-3)
- net *9: now also D1.2 (A)
- net +5V: now also Flex_Sensor1.2 (A1); no longer Flex_Sensor1.1 (VCC)
- net 12: no longer D1.2 (A)
- net A1: now also Flex_Sensor1.1 (VCC); no longer Flex_Sensor1.2 (A1)
- net CLK: now also Encodeur1.3 (SW); no longer Encodeur1.5 (CLK)
- net RXD: now also J5.4 (Tx); no longer J5.5 (Rx)
- net SW: now also Encodeur1.5 (CLK); no longer Encodeur1.3 (SW)
- net TXD: now also J5.5 (Rx); no longer J5.4 (Tx)
- net D3 renamed *3
- net *3: no longer Servo_Moteur1.3 (-3)
Other:
- moved on the sheet: R7

Commit message: V2 de routage de la carte
Connections:
- net 12 is gone; now on net CS: J2.6 (Pin_6)
- net CS: no longer J2.8 (Pin_8)
- net RXD: now also J5.5 (Rx); no longer J5.4 (Tx)
- net TXD: now also J5.4 (Tx); no longer J5.5 (Rx)
- new net *10: J2.8 (Pin_8)
- no-connect marks 10 -> 13
Changed lines of the file:
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@@
 	)
 	(no_connect
+		(at 85.09 67.31)
+	)
+	(no_connect
 		(at 207.01 66.04)
 	)
@@
 	)
 	(no_connect
-		(at 31.75 90.17)
+		(at 193.04 137.16)
 	)
 	(no_connect
-		(at 85.09 62.23)
+		(at 196.85 137.16)
+	)
+	(no_connect
+		(at 31.75 90.17)
 	)
 	(no_connect
@@
 	)
 	(no_connect
+		(at 189.23 137.16)
+	)
+	(no_connect
 		(at 207.01 53.34)
 	)
@@
 		)
 	)
+	(label "7"
+		(at 201.93 60.96 180)
+		(effects
+			(font
+				(size 1.27 1.27)
+			)
+			(justify right bottom)
+		)
+	)
 	(label "*9"
 		(at 161.29 57.15 180)
@@
 		)
 	)
-	(label "7"
-		(at 201.93 63.5 180)
-		(effects
-			(font
-				(size 1.27 1.27)
-			)
-			(justify right bottom)
-		)
-	)
 	(label "12"
 		(at 85.09 62.23 180)
@@
 		)
 	)
-	(label "8"
-		(at 201.93 60.96 180)
-		(effects
-			(font
-				(size 1.27 1.27)
-			)
-			(justify right bottom)
-		)
-	)
 	(label "SDA{slash}A4"
 		(at 137.16 68.58 270)
@@
 		)
 	)
+	(label "8"
+		(at 201.93 63.5 180)
+		(effects
+			(font
+				(size 1.27 1.27)
+			)
+			(justify right bottom)
+		)
+	)
 	(label "SDA{slash}A4"
 		(at 31.75 92.71 0)
@@
 		)
 	)
-	(global_label "CS"
+	(global_label "A1"
 		(shape input)
-		(at 85.09 67.31 0)
+		(at 29.21 173.99 180)
 		(fields_autoplaced yes)
 		(effects
@@
 				(size 1.27 1.27)
 			)
-			(justify left)
+			(justify right)
 		)
 		(property "Intersheetrefs" "${INTERSHEET_REFS}"
-			(at 90.6498 67.31 0)
+			(at 23.8316 173.99 0)
 			(effects
 				(font
 					(size 1.27 1.27)
 				)
-				(justify left)
+				(justify right)
 				(hide yes)
 			)
 		)
 	)
-	(global_label "A1"
+	(global_label "SCL"
 		(shape input)
-		(at 29.21 173.99 180)
+		(at 31.75 95.25 180)
 		(fields_autoplaced yes)
 		(effects
@@
 		)
 		(property "Intersheetrefs" "${INTERSHEET_REFS}"
-			(at 23.8316 173.99 0)
+			(at 25.1621 95.25 0)
 			(effects
 				(font
@@
 		)
 	)
-	(global_label "SCL"
+	(global_label "CS"
 		(shape input)
-		(at 31.75 95.25 180)
+		(at 85.09 62.23 0)
 		(fields_autoplaced yes)
 		(effects
@@
 				(size 1.27 1.27)
 			)
-			(justify right)
+			(justify left)
 		)
 		(property "Intersheetrefs" "${INTERSHEET_REFS}"
-			(at 25.1621 95.25 0)
+			(at 90.6498 62.23 0)
 			(effects
 				(font
 					(size 1.27 1.27)
 				)
-				(justify right)
+				(justify left)
 				(hide yes)
 			)
@@
 		(dnp no)
 		(property "Reference" "LTC1050_1"
-			(at 190.5 132.08 0)
+			(at 192.786 121.412 0)
 			(effects
 				(font
@@
 		)
 		(property "Value" "LTC1050"
-			(at 190.5 134.62 0)
+			(at 192.786 123.952 0)
 			(effects
 				(font
@@
 		(pin "7"
 		)
+		(pin "5"
+		)
+		(pin "1"
+		)
+		(pin "8"
+		)
 		(instances
