File: 1/1.kicad_pcb (KiCad board)
At the start: 2 copper layers, 68.6 x 53.3 mm, 23 parts, among them J1 Power, J2 Digital/PWM, J3 Analog, J4 Digital/PWM, J5 HC-05, U2 LTC1050

Commit message: Modifactions on kicad project and ltspice are added
Parts:
- removed Entree_Sin1: Conn_01x02, Connector_PinSocket_2.54mm:PinSocket_1x02_P2.54mm_Vertical
Connections:
- Capteur1 pad 1: /*5 -> Net-(Capteur1-Pin_1)
- R5 pad 1: /*5 -> Net-(Capteur1-Pin_1)
Routing:
- net GND: track 151.3 -> 120.8 mm
- net /*5: track 13.4 -> 0.00 mm
- net Net-(Capteur1-Pin_1): track 0.00 -> 8.64 mm
- added copper zone on B.Cu, net GND

Commit message: Rajout des capteurs
Connections:
- J5 pad 4: /2 -> /7
- J5 pad 5: /*3 -> /8
Routing:
- net GND: track 120.8 -> 0.96 mm
Changed lines of the file:
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@@
 			(net 14 "/8")
 			(pinfunction "Pin_10")
-			(pintype "passive+no_connect")
+			(pintype "passive")
 		)
 		(embedded_fonts no)
@@
 			(net 15 "/7")
 			(pinfunction "Pin_1")
-			(pintype "passive+no_connect")
+			(pintype "passive")
 		)
 		(pad "2" thru_hole oval
@@
 			(layers "*.Cu" "*.Mask")
 			(remove_unused_layers no)
-			(net 20 "/2")
+			(net 15 "/7")
 			(pinfunction "Tx")
 			(pintype "bidirectional")
@@
 			(layers "*.Cu" "*.Mask")
 			(remove_unused_layers no)
-			(net 24 "/*3")
+			(net 14 "/8")
 			(pinfunction "Rx")
 			(pintype "bidirectional")
@@
 	)
 	(segment
-		(start 150 53.5)
-		(end 151 53.5)
-		(width 1)
-		(layer "B.Cu")
-		(net 1)
-	)
-	(segment
-		(start 125.119 51.381)
-		(end 126.416 50.084)
-		(width 1)
-		(layer "B.Cu")
-		(net 1)
-	)
-	(segment
-		(start 142.801 53.914001)
-		(end 142.801 65.319)
-		(width 1)
-		(layer "B.Cu")
-		(net 1)
-	)
-	(segment
-		(start 151 53.5)
-		(end 154.5 57)
-		(width 1)
-		(layer "B.Cu")
-		(net 1)
-	)
-	(segment
-		(start 148.199 51.699)
-		(end 138.881 51.699)
-		(width 1)
-		(layer "B.Cu")
-		(net 1)
-	)
-	(segment
 		(start 126.416 49.27771)
 		(end 126.416 49.2)
@@
 	)
 	(segment
-		(start 138.881 51.699)
-		(end 140.585999 51.699)
-		(width 1)
-		(layer "B.Cu")
-		(net 1)
-	)
-	(segment
-		(start 130.63829 53.5)
-		(end 126.416 49.27771)
-		(width 1)
-		(layer "B.Cu")
-		(net 1)
-	)
-	(segment
-		(start 157.5 60)
-		(end 154.5 57)
-		(width 1)
-		(layer "B.Cu")
-		(net 1)
-	)
-	(segment
 		(start 126.416 50.084)
 		(end 126.416 49.2)
 		(width 1)
 		(layer "B.Cu")
-		(net 1)
-	)
-	(segment
-		(start 125.119 73.799)
-		(end 125.119 51.381)
-		(width 1)
-		(layer "B.Cu")
-		(net 1)
-	)
-	(segment
-		(start 157.5 91)
-		(end 157.5 60)
-		(width 1)
-		(layer "B.Cu")
-		(net 1)
-	)
-	(segment
-		(start 142.801 65.319)
-		(end 137 71.12)
-		(width 1)
-		(layer "B.Cu")
-		(net 1)
-	)
-	(segment
-		(start 137.08 53.5)
-		(end 130.63829 53.5)
-		(width 1)
-		(layer "B.Cu")
-		(net 1)
-	)
-	(segment
-		(start 137.08 53.5)
-		(end 138.881 51.699)
-		(width 1)
-		(layer "B.Cu")
-		(net 1)
-	)
-	(segment
-		(start 150 53.5)
-		(end 148.199 51.699)
-		(width 1)
-		(layer "B.Cu")
-		(net 1)
-	)
-	(segment
-		(start 140.585999 51.699)
-		(end 142.801 53.914001)
-		(width 1)
-		(layer "B.Cu")
-		(net 1)
-	)
-	(segment
-		(start 127.32 76)
-		(end 125.119 73.799)
-		(width 1)
-		(layer "B.Cu")

Commit message: Face avant v1
Parts:
- removed R2: 1k, Resistor_THT:R_Axial_DIN0207_L6.3mm_D2.5mm_P10.16mm_Horizontal
Connections:
- net /*10 renamed CS
- net /*11 renamed SI
- net /*3 renamed D3
- net /*5 renamed SW
- net /13 renamed SCK
- net /2 renamed CLK
- net /4 renamed DATA
- net /7 renamed TXD
- net /8 renamed RXD
- net /A1 renamed A1
- net /SCL/A5 renamed SCL
- net /SDA/A4 renamed A4
- net Net-(U2-+) renamed R2

Commit message: MAJ de la face arrière avant la routage
Parts:
- added Encodeur1: ~, projet_capteur_artur:Encodeur, F.Cu at (185.5, 102.0)
- added Flex_Sensor1: ~, projet_capteur_artur:flex_sensor, F.Cu at (227.0, 49.9)
- added Potentiomètre3: ~, projet_capteur_artur:potentiometre_digit, F.Cu at (222.7, 72.5)
- added R7: 10k, Resistor_THT:R_Axial_DIN0207_L6.3mm_D2.5mm_P10.16mm_Horizontal, F.Cu at (208.9, 92.6)
- added Servo_Moteur1: ~, projet_capteur_artur:servo, F.Cu at (197.7, 102.0)
- moved Capteur1 97.3 mm to (217.1, 97.0)
- moved U2 93.8 mm to (222.2, 84.2), turned to 0 degrees
- moved C1 90.5 mm to (218.7, 58.1)
- moved R6 89.2 mm to (208.9, 88.6)
- moved D1 88.7 mm to (209.8, 98.4)
- moved J5 82.5 mm to (181.0, 52.8), turned to 0 degrees
- moved C4 82.0 mm to (222.2, 97.9), turned to 0 degrees
- moved R5 81.6 mm to (208.9, 84.5)
- moved R1 71.5 mm to (208.9, 72.4), turned to 0 degrees
- moved C2 64.7 mm to (218.7, 64.6)
- moved R3 62.2 mm to (208.9, 76.4), turned to 0 degrees
- moved R4 59.7 mm to (208.9, 80.5)
- moved U1 38.2 mm to (192.3, 83.1), turned to 0 degrees
Connections:
- D1 pad 2: DATA -> /12
Routing:
- net Net-(C4-Pad1): track 82.2 -> 0.00 mm
- net +5V: track 60.0 -> 0.00 mm
- net R2: track 20.8 -> 0.00 mm
- net Net-(U2--): track 20.6 -> 0.00 mm
- net (no net): track 17.6 -> 0.00 mm
- net SCL: track 15.0 -> 0.00 mm
- net A4: track 15.0 -> 0.22 mm
- net Net-(Capteur1-Pin_1): track 8.64 -> 0.00 mm
- net AmpliOut: track 6.57 -> 0.00 mm
- net Net-(D1-K): track 6.42 -> 0.00 mm
- net GND: track 0.96 -> 0.00 mm

Commit message: Rootage v1
Parts:
- removed MH1, MH2, MH3, MH4: MountingHole_3.2mm, Arduino_MountingHole:MountingHole_3.2mm
- R6: value R -> 320
- moved D1 113.7 mm to (105.5, 53.0), turned to 90 degrees
- moved LTC1050_1 106.4 mm to (115.8, 86.7), turned to -90 degrees
- moved R6 102.6 mm to (112.0, 54.9), turned to -90 degrees
- moved C1 100.8 mm to (118.0, 62.5), turned to -90 degrees
- moved Potent3 89.3 mm to (133.8, 63.3), turned to 180 degrees
- moved Capteur1 88.7 mm to (129.2, 85.0), turned to -90 degrees
- moved R1 88.6 mm to (120.4, 76.5)
- moved C4 87.0 mm to (135.5, 90.8), turned to 90 degrees
- moved J5 81.6 mm to (104.8, 82.0), turned to 90 degrees
- moved R3 79.7 mm to (130.6, 91.0), turned to 180 degrees
- moved R5 79.1 mm to (130.6, 73.5), turned to 180 degrees
- moved Flex_Sensor1 76.5 mm to (160.6, 87.8), turned to 180 degrees
- moved C2 73.5 mm to (148.0, 84.5), turned to -90 degrees
- moved Servo_Moteur1 72.2 mm to (134.5, 67.0)
- moved R4 66.9 mm to (142.0, 81.9), turned to -90 degrees
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- renumbered U2 to LTC1050_1, Potentiomètre3 to Potent3
Connections:
- D1 pad 2: /12 -> /*9
- Encodeur1 pad 3: SW -> CLK
- Encodeur1 pad 5: CLK -> SW
- Flex_Sensor1 pad 1: +5V -> A1
- Flex_Sensor1 pad 2: A1 -> +5V
- J4 pad 5: D3 -> /*3
- J5 pad 4: TXD -> RXD
- J5 pad 5: RXD -> TXD
- Servo_Moteur1 pad 3: D3 -> /*6
Routing:
- net +5V: track 0.00 -> 204.2 mm
- net R2: track 0.00 -> 90.9 mm
- net TXD: track 0.00 -> 59.8 mm, vias 0 -> 2
- net RXD: track 0.00 -> 57.4 mm, vias 0 -> 2
- net Net-(C4-Pad1): track 0.00 -> 45.4 mm
- net /*9: track 0.00 -> 37.9 mm, vias 0 -> 2
- net SCL: track 0.00 -> 35.9 mm
- net A4: track 0.22 -> 31.1 mm
- net /*6: track 0.00 -> 26.1 mm
- net Net-(LTC1050_1--): track 0.00 -> 25.8 mm
- net Net-(Capteur1-Pin_1): track 0.00 -> 24.8 mm
- net CLK: track 0.00 -> 21.1 mm
- net CS: track 0.00 -> 17.6 mm
- net DATA: track 0.00 -> 16.5 mm
- net SCK: track 0.00 -> 16.3 mm
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Other:
- board size 68.6 x 53.3 mm -> 69.2 x 53.3 mm

Commit message: V2 de routage de la carte
Parts:
- moved J5 60.4 mm to (152.5, 45.0), turned to -90 degrees
- moved R7 39.4 mm to (123.9, 107.0), turned to 0 degrees
- moved Encodeur1 38.1 mm to (181.9, 61.1), turned to -90 degrees
- moved D1 33.4 mm to (138.8, 56.1)
- moved C4 32.3 mm to (111.0, 69.8), turned to -90 degrees
- moved R6 27.4 mm to (139.0, 59.5)
- moved R5 27.0 mm to (110.9, 92.0), turned to 0 degrees
- moved R3 26.8 mm to (117.0, 67.9), turned to -90 degrees
- moved C2 23.4 mm to (140.0, 106.5), turned to 0 degrees
- moved C1 22.1 mm to (115.5, 84.5), turned to 0 degrees
- moved Capteur1 21.6 mm to (112.0, 98.0), turned to 90 degrees
- moved Flex_Sensor1 20.8 mm to (151.7, 106.6), turned to 90 degrees
- moved U1 17.7 mm to (162.2, 98.3), turned to 180 degrees
- moved Servo_Moteur1 16.8 mm to (149.0, 58.5), turned to 90 degrees
- moved LTC1050_1 14.3 mm to (125.7, 76.3), turned to 90 degrees
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Connections:
- J2 pad 6: /12 -> CS
- J2 pad 8: CS -> /*10
- J5 pad 4: RXD -> TXD
- J5 pad 5: TXD -> RXD
- LTC1050_1 pad 1: (no net) -> unconnected-(LTC1050_1-GND-Pad1)
- LTC1050_1 pad 5: (no net) -> unconnected-(LTC1050_1-GND-Pad5)
- LTC1050_1 pad 8: (no net) -> unconnected-(LTC1050_1-GND-Pad8)
Routing:
- net +5V: track 204.2 -> 331.2 mm
- net TXD: track 59.8 -> 4.53 mm, vias 2 -> 0
- net RXD: track 57.4 -> 4.50 mm, vias 2 -> 0
- net /*9: track 37.9 -> 4.47 mm, vias 2 -> 0
- net R2: track 90.9 -> 58.8 mm
- net SW: track 13.0 -> 39.5 mm
- net SCL: track 35.9 -> 12.8 mm
- net DATA: track 16.5 -> 35.8 mm
- net /*6: track 26.1 -> 7.07 mm
- net Net-(Capteur1-Pin_1): track 24.8 -> 6.43 mm
- net A4: track 31.1 -> 12.8 mm
- net A1: track 14.5 -> 30.4 mm
- net CS: track 17.6 -> 5.45 mm
- net Net-(C4-Pad1): track 45.4 -> 57.6 mm
- net SCK: track 16.3 -> 5.01 mm
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Other:
- board outline removed
- board text removed: "ICSP"

Commit message: Routage V3
Other:
- board text added: "Maëlys CHRISTIEN Artur NERSISYAN"
Changed lines of the file:
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@@
+		)
+	)
+	(gr_text "Maëlys CHRISTIEN\nArtur  NERSISYAN"
+		(at 185 91 90)
+		(layer "B.Cu" knockout)
+		(effects
+			(font
+				(size 1.5 1.5)
+				(thickness 0.3)
+				(bold yes)
+			)
+			(justify left bottom mirror)
 		)
 	)
